Commit message: change collitions

File: alfredr1/urdf/body_r1.urdf.xacro (robot description, xacro)
@@ -20,5 +20,5 @@
         <origin xyz="0.0325 0 0.049" rpy="0 0 0"/>
         <geometry>
-          <mesh filename="package://alfredr1/urdf/meshes/waist_roll_link.STL"/>
+            <box size="0.061842 0.080477 0.078131" />
         </geometry>
       </collision>
@@ -38,7 +38,7 @@
       </visual>
       <collision>
-        <origin xyz="0 0 0" rpy="0 0 0"/>
+        <origin xyz="0 0 0.123721" rpy="0 0 0"/>
         <geometry>
-          <mesh filename="package://alfredr1/urdf/meshes/waist_yaw_link.STL"/>
+          <box size="0.127992 0.138076 0.245606" />
         </geometry>
       </collision>

File: alfredr1/urdf/head_r1.urdf.xacro (robot description, xacro)
@@ -18,7 +18,7 @@
             </visual>
             <collision>
-                <origin xyz="0 0 0" rpy="0 0 0"/>
+                <origin xyz="0 -0.031688 0.051001" rpy="0 0 0"/>
                 <geometry>
-                    <mesh filename="package://alfredr1/urdf/meshes/head_pitch_link.STL"/>
+                   <box size="0.061441 0.061441 0.157445" />
                 </geometry>
             </collision>
@@ -38,7 +38,7 @@
             </visual>
             <collision>
-                <origin xyz="0 0 0" rpy="0 0 0"/>
+                <origin xyz="0.019307 0 -0.012286" rpy="0 2.891 0"/>
                 <geometry>
-                    <mesh filename="package://alfredr1/urdf/meshes/head_yaw_link.STL"/>
+                    <box size="0.082445 0.087838 0.144796" />
                 </geometry>
             </collision>

File: alfredr1/urdf/r1_urdf.urdf.xacro (robot description, xacro)
@@ -23,7 +23,7 @@
         </visual>
         <collision>
-            <origin xyz="0 0 0" rpy="0 0 0"/>
+            <origin xyz="0.024748 0 -0.067283" rpy="0 0 0"/>
             <geometry>
-                <mesh filename="package://alfredr1/urdf/meshes/pelvis_link.STL"/>
+                <box size="0.104 0.104 0.1" />
             </geometry>
         </collision>
